File: HardwareKiCad/v1/GPSWatch.kicad_sch (KiCad schematic)
At the start: 53 parts, among them IC2 BMA423, J1 Battery, J2 USB_B_Micro, J4 Micro_SD_Card_Det2, J5 Conn_01x04_Pin, SW1 SW_SPDT, SW3 SW_Push, SW4 SW_Push, SW5 SW_Push, U1 L96-M33, U2 STM32L476RGTx, U3 PES12-40S-N0024, U4 MCP73871, Y2 ABS07-32.768KHZ-6-T, Y3 ABM3-8.000MHZ-B4Y-T

Commit message: Add version 1.1 hardware
Other:
- note added: "07/21/2025"
Changed lines of the file:
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@@
 		)
 	)
+	(text "07/21/2025"
+		(exclude_from_sim no)
+		(at 212.344 193.548 0)
+		(effects
+			(font
+				(size 1.27 1.27)
+				(color 170 29 29 1)
+			)
+		)
+	)
 	(text "to do:\nconnect ep to gnd \nw/ ground pour that vias to gnd plane"
 		(exclude_from_sim no)
@@
 		(dnp no)
 		(property "Reference" "SW4"
-			(at 78.486 118.11 0)
+			(at 74.93 122.174 0)
 			(effects
 				(font
