File: Hardware/v1.1/GPSWatch.kicad_pcb (KiCad board)
At the start: 2 copper layers, 41 x 42 mm, 58 parts, among them J1 USB_B_Micro, J2 Battery, J4 Micro_SD_Card_Det2, J5 Conn_01x04_Pin, SW1 EC05E1220401, SW2 SW_SPDT, SW3 SW_Push, SW4 SW_Push, SW5 SW_Push, U1 STM32F103C8Tx, U2 AMS1117-3.3, U3 MCP73831-2-OT, U4 TPS2116DRL, U5 L96-M33, U6 BMA456, Y1 ABM3-8.000MHZ-B4Y-T

Commit message: Add hardware v1.1 to repository
Parts:
- removed C11: 100uF, Capacitor_SMD:C_0603_1608Metric
- removed C14: 0.1uF, Capacitor_SMD:C_0402_1005Metric
- C12: value 0.1uF -> 10uF
- C13: value 4.7uF -> 22uF
Routing:
- net GND: track 122.4 -> 119.3 mm, vias 51 -> 50
