File: Hardware/v1.1/GPSWatch.kicad_sch (KiCad schematic)
At the start: 58 parts, among them J1 USB_B_Micro, J2 Battery, J4 Micro_SD_Card_Det2, J5 Conn_01x04_Pin, SW1 EC05E1220401, SW2 SW_SPDT, SW3 SW_Push, SW4 SW_Push, SW5 SW_Push, U1 STM32F103C8Tx, U2 AMS1117-3.3, U3 MCP73831-2-OT, U4 TPS2116DRL, U5 L96-M33, U6 BMA456, Y1 ABM3-8.000MHZ-B4Y-T

Commit message: Add hardware v1.1 to repository
Parts:
- removed C11: 100uF, Capacitor_SMD:C_0603_1608Metric, symbol Device:C
- removed C14: 0.1uF, Capacitor_SMD:C_0402_1005Metric, symbol Device:C
- C12: value 0.1uF -> 10uF; footprint Capacitor_SMD:C_0402_1005Metric -> Capacitor_SMD:C_0603_1608Metric
- C13: value 4.7uF -> 22uF
- C22, C7, C8: footprint Capacitor_SMD:C_0402_1005Metric -> Capacitor_SMD:C_0603_1608Metric
Changed lines of the file:
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@@
 	)
 	(junction
-		(at 59.69 99.06)
-		(diameter 0)
-		(color 0 0 0 0)
-	)
-	(junction
 		(at 66.04 124.46)
 		(diameter 0)
@@
 	)
 	(junction
-		(at 38.1 99.06)
-		(diameter 0)
-		(color 0 0 0 0)
-	)
-	(junction
 		(at 36.83 22.86)
 		(diameter 0)
@@
 	)
 	(junction
-		(at 30.48 90.17)
-		(diameter 0)
-		(color 0 0 0 0)
-	)
-	(junction
 		(at 214.63 25.4)
 		(diameter 0)
@@
 	)
 	(junction
-		(at 67.31 90.17)
-		(diameter 0)
-		(color 0 0 0 0)
-	)
-	(junction
 		(at 74.93 166.37)
 		(diameter 0)
@@
 	(wire
 		(pts
-			(xy 67.31 99.06) (xy 67.31 97.79)
-		)
-		(stroke
-			(width 0)
-			(type default)
-		)
-	)
-	(wire
-		(pts
 			(xy 229.87 25.4) (xy 229.87 43.18)
 		)
@@
 	(wire
 		(pts
-			(xy 59.69 99.06) (xy 67.31 99.06)
-		)
-		(stroke
-			(width 0)
-			(type default)
-		)
-	)
-	(wire
-		(pts
 			(xy 52.07 22.86) (xy 52.07 26.67)
 		)
@@
 	(wire
 		(pts
-			(xy 30.48 99.06) (xy 30.48 97.79)
-		)
-		(stroke
-			(width 0)
-			(type default)
-		)
-	)
-	(wire
-		(pts
 			(xy 219.71 156.21) (xy 219.71 143.51)
 		)
@@
 	(wire
 		(pts
-			(xy 59.69 90.17) (xy 67.31 90.17)
+			(xy 59.69 90.17) (xy 71.12 90.17)
 		)
 		(stroke
@@
 	(wire
 		(pts
-			(xy 27.94 90.17) (xy 30.48 90.17)
-		)
-		(stroke
-			(width 0)
-			(type default)
-		)
-	)
-	(wire
-		(pts
 			(xy 205.74 41.91) (xy 207.01 41.91)
 		)
@@
 	(wire
 		(pts
-			(xy 71.12 90.17) (xy 67.31 90.17)
-		)
-		(stroke
-			(width 0)
-			(type default)
-		)
-	)
-	(wire
-		(pts
 			(xy 260.35 149.86) (xy 256.54 149.86)
 		)
@@
 	(wire
 		(pts
-			(xy 30.48 90.17) (xy 38.1 90.17)
+			(xy 27.94 90.17) (xy 38.1 90.17)
 		)
 		(stroke
@@
 	(wire
 		(pts
-			(xy 30.48 99.06) (xy 38.1 99.06)
-		)
-		(stroke
-			(width 0)
-			(type default)
-		)
-	)
-	(wire
-		(pts
 			(xy 195.58 45.72) (xy 200.66 45.72)
 		)
@@
 	(symbol
 		(lib_id "Device:C")
-		(at 67.31 93.98 0)
-		(unit 1)
-		(exclude_from_sim no)
-		(in_bom yes)
-		(on_board yes)
-		(dnp no)
-		(property "Reference" "C14"
-			(at 68.072 91.948 0)
-			(effects
-				(font
-					(size 1.27 1.27)
-				)
-				(justify left)
-			)
-		)
-		(property "Value" "0.1uF"
-			(at 68.326 96.52 0)
-			(effects
-				(font
-					(size 1.27 1.27)
-				)
-				(justify left)
-			)
-		)
-		(property "Footprint" "Capacitor_SMD:C_0402_1005Metric"
-			(at 68.2752 97.79 0)
-			(effects
-				(font
-					(size 1.27 1.27)
-				)
-				(hide yes)
-			)
-		)
-		(property "Datasheet" "~"
-			(at 67.31 93.98 0)
-			(effects
-				(font
-					(size 1.27 1.27)
-				)
-				(hide yes)
-			)
-		)
-		(property "Description" "Unpolarized capacitor"
-			(at 67.31 93.98 0)
-			(effects
-				(font
-					(size 1.27 1.27)
-				)
-				(hide yes)
-			)
-		)
-		(pin "1"
-		)
-		(pin "2"
-		)
-		(instances
-			(project "GPSWatch"
-				(path "/9f4df342-8db3-41c4-bd1d-44c5477f93e2"
-					(reference "C14")
-					(unit 1)
-				)
-			)
-		)
-	)
-	(symbol
-		(lib_id "Device:C")
 		(at 222.25 29.21 0)
 		(unit 1)
@@
 			)
 		)
-		(property "Footprint" "Capacitor_SMD:C_0402_1005Metric"
+		(property "Footprint" "Capacitor_SMD:C_0603_1608Metric"
 			(at 254.9652 33.02 0)
 			(effects
@@
 			)
 		)
-		(property "Value" "4.7uF"
+		(property "Value" "22uF"
 			(at 60.706 96.52 0)
 			(effects
@@
 	(symbol
 		(lib_id "Device:C")
-		(at 30.48 93.98 0)
-		(unit 1)
-		(exclude_from_sim no)
-		(in_bom yes)
-		(on_board yes)
-		(dnp no)
-		(property "Reference" "C11"
-			(at 31.242 91.948 0)
-			(effects
-				(font
-					(size 1.27 1.27)
-				)
-				(justify left)
-			)
-		)
-		(property "Value" "100uF"
-			(at 31.496 96.52 0)
-			(effects
-				(font
-					(size 1.27 1.27)
-				)
-				(justify left)
-			)
-		)
-		(property "Footprint" "Capacitor_SMD:C_0603_1608Metric"
-			(at 31.4452 97.79 0)
-			(effects
-				(font
-					(size 1.27 1.27)
-				)
-				(hide yes)
-			)
-		)
-		(property "Datasheet" "~"
-			(at 30.48 93.98 0)
-			(effects
-				(font
-					(size 1.27 1.27)
-				)
-				(hide yes)
-			)
-		)
-		(property "Description" "Unpolarized capacitor"
-			(at 30.48 93.98 0)
-			(effects
-				(font
-					(size 1.27 1.27)
-				)
-				(hide yes)
-			)
-		)
-		(pin "1"
-		)
-		(pin "2"
-		)
-		(instances
-			(project ""
-				(path "/9f4df342-8db3-41c4-bd1d-44c5477f93e2"
-					(reference "C11")
-					(unit 1)
-				)
-			)
-		)
-	)
-	(symbol
-		(lib_id "Device:C")
 		(at 160.02 76.2 0)
 		(unit 1)
@@
 			)
 		)
-		(property "Footprint" "Capacitor_SMD:C_0402_1005Metric"
+		(property "Footprint" "Capacitor_SMD:C_0603_1608Metric"
 			(at 160.9852 80.01 0)
 			(effects
@@
 			)
 		)
-		(property "Footprint" "Capacitor_SMD:C_0402_1005Metric"
+		(property "Footprint" "Capacitor_SMD:C_0603_1608Metric"
 			(at 272.7452 33.02 0)
 			(effects
@@
 			)
 		)
-		(property "Value" "0.1uF"
+		(property "Value" "10uF"
 			(at 39.116 96.52 0)
 			(effects
@@
 			)
 		)
-		(property "Footprint" "Capacitor_SMD:C_0402_1005Metric"
+		(property "Footprint" "Capacitor_SMD:C_0603_1608Metric"
 			(at 39.0652 97.79 0)
 			(effects
